Commit message: updates to the urdf file

File: Drone_Model/urdf/Drone_Model.urdf (robot description, URDF)
Before this commit: robot FULL_ASSEM_0802_ForInsert, 5 links, 4 joints
Joints:
- removed joint Revolute_73
- removed joint Revolute_74
- removed joint Revolute_75
- removed joint Revolute_76
- added joint Front-Left-Joint: type continuous, parent base_link, child Propeller_CW_Puller_2, origin xyz=-0.109217294 -0.0793510091 0.029 rpy=0 0 0, axis 0 0 -1
- added joint Front-Right-Joint: type continuous, parent base_link, child Propeller_CCW_Puller_1, origin xyz=0.109217294 -0.0793510091 0.029 rpy=0 0 0, axis 0 0 -1
- added joint Rear-Left-Joint: type continuous, parent base_link, child Propeller_CCW_Puller_2, origin xyz=-0.109217294 0.0793510091 0.029 rpy=0 0 0, axis 0 0 -1
- added joint Rear-Right-Joint: type continuous, parent base_link, child Propeller_CW_Puller_1, origin xyz=0.109217294 0.0793510091 0.029 rpy=0 0 0, axis 0 0 -1
